Commit message: Now all is working including Moveit

File: ers6_ws/src/hardware/urdf/ers6_robot.urdf (robot description, URDF)
Before this commit: robot ers6, 7 links, 6 joints
Links:
- removed link link1
- removed link link2
- removed link link3
- removed link link4
- removed link link5
- removed link link6
- added link a0, mass 1; collision mesh filename=package://ers6_description/meshes/a0.stl scale=0.001 0.001 0.001; visual mesh filename=package://ers6_description/meshes/a0.stl scale=0.005 0.005 0.005
- added link a1, mass 1; collision mesh filename=package://ers6_description/meshes/a1.stl scale=0.001 0.001 0.001; visual mesh filename=package://ers6_description/meshes/a1.stl scale=0.005 0.005 0.005
- added link a2, mass 1; collision mesh filename=package://ers6_description/meshes/a2.stl scale=0.001 0.001 0.001; visual mesh filename=package://ers6_description/meshes/a2.stl scale=0.005 0.005 0.005
- added link a3, mass 1; collision mesh filename=package://ers6_description/meshes/a3.stl scale=0.001 0.001 0.001; visual mesh filename=package://ers6_description/meshes/a3.stl scale=0.005 0.005 0.005
- added link a4, mass 1; collision mesh filename=package://ers6_description/meshes/a4.stl scale=0.001 0.001 0.001; visual mesh filename=package://ers6_description/meshes/a4.stl scale=0.005 0.005 0.005
- added link a5, mass 1; collision mesh filename=package://ers6_description/meshes/a5.stl scale=1 1 1; visual mesh filename=package://ers6_description/meshes/a5.stl scale=0.005 0.005 0.005
- added link world
- link base_link: mass None -> 1; geometry collision mesh filename=package://ers6_description/meshes/Base.stl scale=1 1 1; visual mesh filename=package://ers6_description/meshes/Base.stl scale=0.005 0.005 0.005
Joints:
- added joint base_joint: type fixed, parent world, child base_link, origin xyz=0 0 0 rpy=0 0 0
- joint a1_to_a0: axis 1 0 0 -> 0 0 1; child link6 -> a0; limit lower=-2.62 upper=2.62 effort=5 velocity=3 -> lower=-1 upper=1 effort=1000 velocity=0.5; origin xyz=0 0 0 rpy=0 0 0 -> xyz=0 0 0.1 rpy=0 0 0; parent link5 -> a1
- joint a2_to_a1: child link5 -> a1; limit lower=-2.62 upper=2.62 effort=5 velocity=3 -> lower=-1 upper=1 effort=1000 velocity=0.5; origin xyz=0 0 0 rpy=0 0 0 -> xyz=0 0 0.1 rpy=0 0 0; parent link4 -> a2
- joint a3_to_a2: child link4 -> a2; limit lower=-2.62 upper=2.62 effort=5 velocity=3 -> lower=-1 upper=1 effort=1000 velocity=0.5; origin xyz=0 0 0 rpy=0 0 0 -> xyz=0 0 0.1 rpy=0 0 0; parent link3 -> a3
- joint a4_to_a3: axis 1 0 0 -> 0 -1 0.0032; child link3 -> a3; limit lower=-2.62 upper=2.62 effort=5 velocity=3 -> lower=-1 upper=1 effort=1000 velocity=0.5; origin xyz=0 0 0 rpy=0 0 0 -> xyz=0 0 0.1 rpy=0 0 0; parent link2 -> a4
- joint a5_to_a4: axis 0 1 0 -> 0 0 1; child link2 -> a4; limit lower=-2.62 upper=2.62 effort=5 velocity=3 -> lower=-1 upper=1 effort=1000 velocity=0.5; origin xyz=0 0 0 rpy=0 0 0 -> xyz=0 0 0.1 rpy=0 0 0; parent link1 -> a5
- joint base_link_to_a5: child link1 -> a5; limit lower=-2.62 upper=2.62 effort=5 velocity=3 -> lower=-1 upper=1 effort=1000 velocity=0.5; origin xyz=0 0 0 rpy=0 0 0 -> xyz=10 5 0 rpy=3.1416 0 0
