Commit message: Limit J4 to its real range (0 to 0.8 rad)
Measured on the arm: the J4 servo only covers ~95 deg over 500-2500 us
and hits an end stop at the software zero, giving a usable range of
about 0-47 deg. Update both URDFs and MoveIt's joint_limits.yaml so
neither the controller nor MoveIt commands J4 outside that range.

Co-Authored-By: Claude Opus 5.5 <noreply@anthropic.com>
Claude-Session: https://claude.ai/code/session_01FPkvXy1keLMXnn1W2BJoi6

File: ers_3_ws/src/description/urdf/ers6.urdf (robot description, URDF)
Before this commit: robot ers6, 8 links, 7 joints
Joints:
- joint Joint_4: limit lower=-1.5708 upper=1.5708 effort=1000 velocity=2.0 -> lower=0.0 upper=0.8 effort=1000 velocity=2.0
